Commit message: Ran in Gazebo

File: urdf_final/urdf/urdf_final.urdf (robot description, URDF)
Before this commit: robot urdf_final, 5 links, 4 joints
Links:
- removed link back_left_wheel
- removed link back_right_wheel
- removed link front_left_wheel
- removed link front_right_wheel
- added link back_left_wheel_link, mass 0.049871; collision mesh filename=file://$(find robot_package)/urdf_final/meshes/back_left_wh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; visual mesh filename=file://$(find robot_package)/urdf_final/meshes/back_left_wh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
- added link back_right_wheel_link, mass 0.049871; collision mesh filename=file://$(find robot_package)/urdf_final/meshes/back_right_w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; visual mesh filename=file://$(find robot_package)/urdf_final/meshes/back_right_w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
- added link front_left_wheel_link, mass 0.049871; collision mesh filename=file://$(find robot_package)/urdf_final/meshes/front_left_w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; visual mesh filename=file://$(find robot_package)/urdf_final/meshes/front_left_w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
- added link front_right_wheel_link, mass 0.049871; collision mesh filename=file://$(find robot_package)/urdf_final/meshes/front_right_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; visual mesh filename=file://$(find robot_package)/urdf_final/meshes/front_right_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
- link chasis: geometry collision mesh filename=file://$(find robot_package)/urdf_final/meshes/chasis.STL; visual mesh filename=file://$(find robot_package)/urdf_final/meshes/chasis.STL
Joints:
- removed joint back_left_wheel
- removed joint back_right_wheel
- removed joint front_left_wheel
- removed joint front_right_wheel
- added joint back_left_wheel_joint: type continuous, parent chasis, child back_left_wheel_link, origin xyz=0.1175 -0.113 -0.03 rpy=-1.5708 -1.0094 3.1416, axis 0 0 1, limit lower=-3.14 upper=3.14 effort=200 velocity=5
- added joint back_right_wheel_joint: type continuous, parent chasis, child back_right_wheel_link, origin xyz=0.1175 0.113 -0.03 rpy=1.5708 -0.55618 3.1416, axis 0 0 1, limit lower=-3.14 upper=3.14 effort=200 velocity=5
- added joint front_left_wheel_joint: type continuous, parent chasis, child front_left_wheel_link, origin xyz=-0.1175 -0.113 -0.03 rpy=-1.5708 1.3416 3.1416, axis 0 0 1, limit lower=-3.14 upper=3.14 effort=200 velocity=5
- added joint front_right_wheel_joint: type continuous, parent chasis, child front_right_wheel_link, origin xyz=-0.1175 0.113 -0.03 rpy=1.5708 0.55618 3.1416, axis 0 0 1, limit lower=-3.14 upper=3.14 effort=200 velocity=5
