Commit message: Added launching the world with the robot

File: urdf/urdf/urdf_final.urdf (robot description, URDF)
Before this commit: robot urdf_final, 5 links, 4 joints
Links:
- link back_left_wheel_link: geometry collision mesh filename=file://$(find robot_package)/urdf/meshes/back_left_wheel.STL; visual mesh filename=file://$(find robot_package)/urdf/meshes/back_left_wheel.STL
- link back_right_wheel_link: geometry collision mesh filename=file://$(find robot_package)/urdf/meshes/back_right_wheel.S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; visual mesh filename=file://$(find robot_package)/urdf/meshes/back_right_wheel.S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
- link chasis: geometry collision mesh filename=file://$(find robot_package)/urdf/meshes/chasis.STL; visual mesh filename=file://$(find robot_package)/urdf/meshes/chasis.STL
- link front_left_wheel_link: geometry collision mesh filename=file://$(find robot_package)/urdf/meshes/front_left_wheel.S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; visual mesh filename=file://$(find robot_package)/urdf/meshes/front_left_wheel.S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
- link front_right_wheel_link: geometry collision mesh filename=file://$(find robot_package)/urdf/meshes/front_right_wheel.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; visual mesh filename=file://$(find robot_package)/urdf/meshes/front_right_wheel.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
