Commit message: Included the robot drive

File: description/urdf/gazebo.xacro (robot description, xacro)
@@ -1,19 +1,4 @@
 <?xml version="1.0"?>
 <robot xmlns:xacro="http://www.ros.org/wiki/xacro">
-    <gazebo reference="chasis">
-        <material>Gazebo/Green</material>
-    </gazebo>
-    <gazebo reference="back_right_wheel_link">
-        <material>Gazebo/Blue</material>
-    </gazebo>
-    <gazebo reference="back_left_wheel_link">
-        <material>Gazebo/Blue</material>
-    </gazebo>
-    <gazebo reference="front_right_wheel_link">
-        <material>Gazebo/Blue</material>
-    </gazebo>
-    <gazebo reference="front_left_wheel_link">
-        <material>Gazebo/Blue</material>
-    </gazebo>
     <gazebo>
         <plugin name="gazebo_ros_joint_state_publisher"
@@ -34,5 +19,5 @@
     </gazebo>
     <joint name="camera_optical_joint" type="fixed">
-        <origin xyz="0 0 0" rpy="0 0 0" />
+        <origin xyz="-0.25 0 0" rpy="0 0 ${math.pi}" />
         <parent link="chasis" />
         <child link="camera_link" />
@@ -40,6 +25,6 @@
     <link name="camera_link"></link>
     <gazebo reference="camera_link">
-        <sensor type="depth" name="my_camera">
-            <update_rate>9</update_rate>
+        <sensor type="camera" name="my_camera">
+            <update_rate>20</update_rate>
             <visualize>true</visualize>
             <camera name="cam">
@@ -48,5 +33,5 @@
                     <width>640</width>
                     <height>480</height>
-                    <format>R8B8G8</format>
+                    <format>RGB8</format>
                 </image>
                 <clip>

File: description/urdf/urdf_final.urdf (robot description, URDF)
Before this commit: robot Mecanum_robot, 5 links, 4 joints
Links:
- added link base_link
- link back_left_wheel_link: geometry collision mesh filename=file://$(find robot_package)/description/meshes/back_left_w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; visual mesh filename=file://$(find robot_package)/description/meshes/back_left_w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
- link back_right_wheel_link: geometry collision mesh filename=file://$(find robot_package)/description/meshes/back_right_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; visual mesh filename=file://$(find robot_package)/description/meshes/back_right_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
- link chasis: geometry collision mesh filename=file://$(find robot_package)/description/meshes/chasis.STL; visual mesh filename=file://$(find robot_package)/description/meshes/chasis.STL
- link front_left_wheel_link: geometry collision mesh filename=file://$(find robot_package)/description/meshes/front_left_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; visual mesh filename=file://$(find robot_package)/description/meshes/front_left_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
- link front_right_wheel_link: geometry collision mesh filename=file://$(find robot_package)/description/meshes/front_right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; visual mesh filename=file://$(find robot_package)/description/meshes/front_right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
Joints:
- added joint chasis_joint: type fixed, parent base_link, child chasis, origin xyz=0 0 0 rpy=0 0 ${math.pi}
