Commit message: Depth and RGB camera added

File: description/urdf/gazeboDepthCamera.xacro (robot description, xacro)
@@ -14,5 +14,5 @@
     </link>
     <joint name="camera_optical_joint" type="fixed">
-        <origin xyz="0 0 0" rpy="${-math.pi/2} 0 ${-math.pi/22}" />
+        <origin xyz="0 0 0" rpy="${-math.pi/2} 0 ${-math.pi/2}" />
         <parent link="camera_link" />
         <child link="camera_link_optical" />
@@ -21,14 +21,13 @@
     <gazebo reference="camera_link">
         <material>Gazebo/Red</material>
-        <sensor name="camera" type="camera">
-            <pose> 0 0 0 0 0 0 </pose>
+        <sensor type="depth" name="my_camera">
+            <update_rate>20</update_rate>
             <visualize>true</visualize>
-            <update_rate>10</update_rate>
-            <camera>
+            <camera name="cam">
                 <horizontal_fov>1.089</horizontal_fov>
                 <image>
-                    <format>R8G8B8</format>
                     <width>640</width>
                     <height>480</height>
+                    <format>B8G8R8</format>
                 </image>
                 <clip>
@@ -36,7 +35,14 @@
                     <far>8.0</far>
                 </clip>
+                <noise>
+                    <type>gaussian</type>
+                    <mean>0.0</mean>
+                    <stddev>0.007</stddev>
+                </noise>
             </camera>
             <plugin name="camera_controller" filename="libgazebo_ros_camera.so">
                 <frame_name>camera_link_optical</frame_name>
+                <min_depth>0.1</min_depth>
+                <max_depth>500</max_depth>
             </plugin>
         </sensor>

File: description/urdf/gazeboTransforms_update.xacro (robot description, xacro)
@@ -5,5 +5,5 @@
             filename="libgazebo_ros_joint_state_publisher.so">
             <update_rate>20</update_rate>
-            <joint_name>chasis</joint_name>
+            <joint_name>chasis_joint</joint_name>
             <joint_name>back_right_wheel_joint</joint_name>
             <joint_name>back_left_wheel_joint</joint_name>

File: description/urdf/urdf_final.urdf (robot description, URDF)
Before this commit: robot Mecanum_robot, 6 links, 5 joints
Joints:
- joint chasis_joint: origin xyz=0 0 0 rpy=0 0 ${math.pi} -> xyz=0 0 0 rpy=0 0 0
