Commit message: changed to jazzy

File: description/urdf/gazeboLidar.xacro (robot description, xacro)
@@ -1,61 +1,65 @@
 <?xml version="1.0"?>
 <robot xmlns:xacro="http://www.ros.org/wiki/xacro">
-    <xacro:macro name="inertial_cylinder" params="mass length radius *origin">
-        <inertial>
-            <xacro:insert_block name="origin"/>
-            <mass value="${mass}" />
-            <inertia ixx="${(1/12) * mass * (3*radius*radius + length*length)}" ixy="0.0" ixz="0.0"
-                    iyy="${(1/12) * mass * (3*radius*radius + length*length)}" iyz="0.0"
-                    izz="${(1/2) * mass * (radius*radius)}" />
-        </inertial>
-    </xacro:macro>
-    <joint name="lidar_joint" type="fixed">
-        <origin xyz="0 0 0" rpy="0 0 0" />
-        <parent link="chasis" />
-        <child link="lidar_frame" />
-    </joint>
-    <link name="lidar_frame">
-        <visual>
-            <geometry>
-                <cylinder radius="0.05" length="0.04"/>
-                <material name="brown" />
-            </geometry>
-        </visual>
-        <collision>
-            <geometry>
-                <cylinder radius="0.05" length="0.04"/>
-            </geometry>
-        </collision>
-        <xacro:inertial_cylinder mass="0.1" length="0.04" radius="0.05">
-            <origin xyz="0 0 0" rpy="0 0 0"/>
-        </xacro:inertial_cylinder>
-    </link>
-    <gazebo reference="lidar_frame">
-        <material>Gazebo/Red</material>
-        <sensor name="laser" type="ray">
-            <pose> 0 0 0 0 0 0 </pose>
-            <visualize>true</visualize>
-            <update_rate>10</update_rate>
-            <ray>
-                <scan>
-                    <horizontal>
-                        <samples>360</samples>
-                        <min_angle>-3.14</min_angle>
-                        <max_angle>3.14</max_angle>
-                    </horizontal>
-                </scan>
-                <range>
-                    <min>0.3</min>
-                    <max>12</max>
-                </range>
-            </ray>
-            <plugin name="laser_controller" filename="libgazebo_ros_ray_sensor.so">
-                <ros>
-                    <argument>~/out:=scan</argument>
-                </ros>
-                <output_type>sensor_msgs/LaserScan</output_type>
-                <frame_name>laser_frame</frame_name>
-            </plugin>
-        </sensor>
-    </gazebo>
+  <xacro:macro name="inertial_cylinder" params="mass length radius *origin">
+      <inertial>
+          <xacro:insert_block name="origin"/>
+          <mass value="${mass}" />
+          <inertia ixx="${(1/12) * mass * (3*radius*radius + length*length)}" ixy="0.0" ixz="0.0"
+                  iyy="${(1/12) * mass * (3*radius*radius + length*length)}" iyz="0.0"
+                  izz="${(1/2) * mass * (radius*radius)}" />
+      </inertial>
+  </xacro:macro>
+  <joint name="lidar_joint" type="fixed">
+      <origin xyz="0 0 0" rpy="0 0 0" />
+      <parent link="chasis" />
+      <child link="lidar_frame" />
+  </joint>
+  <link name="lidar_frame">
+      <visual>
+          <geometry>
+              <cylinder radius="0.05" length="0.04"/>
+              <material name="brown" />
+          </geometry>
+      </visual>
+      <collision>
+          <geometry>
+              <cylinder radius="0.05" length="0.04"/>
+          </geometry>
+      </collision>
+      <xacro:inertial_cylinder mass="0.1" length="0.04" radius="0.05">
+          <origin xyz="0 0 0" rpy="0 0 0"/>
+      </xacro:inertial_cylinder>
+  </link>
+  <gazebo>
+    <sensor name="lidar_head_link" type="gpu_lidar">
+      <update_rate>30</update_rate>
+      <lidar>
+        <scan>
+          <horizontal>
+            <samples>2800</samples>
+            <resolution>1</resolution>
+            <min_angle>-3.14</min_angle>
+            <max_angle>3.14</max_angle>
+          </horizontal>
+          <vertical>
+            <samples>1</samples>
+            <resolution>0.1</resolution>
+            <min_angle>0.0</min_angle>
+            <max_angle>0.0</max_angle>
+          </vertical>
+        </scan>
+        <range>
+          <min>0.2</min>
+          <max>30.0</max>
+          <resolution>0.01</resolution>
+        </range>
+      </lidar>
+      <always_on>true</always_on>
+      <visualize>true</visualize>
+      <pose>0 0 0.1 0 0 0</pose>  <!-- Adjust pose as needed -->
+    </sensor>
+    <plugin filename="gz-sim-sensors-system" name="gz::sim::systems::Sensors">
+      <render_engine>ogre2</render_engine>
+    </plugin>
+  </gazebo>
 </robot>

File: description/urdf/material.xacro (robot description, xacro)
@@ -1,19 +1,18 @@
 <?xml version="1.0"?>
-<robot
-  xmlns:xacro="http://www.ros.org/wiki/xacro">
+<robot xmlns:xacro="http://www.ros.org/wiki/xacro">
   <material name="red">
-  	<color rgba="1 0 0 1"/>
+    <color rgba="1 0 0 1"/>
   </material>
   <material name="blue">
-  	<color rgba="0 0 1 1"/>
+    <color rgba="0 0 1 1"/>
   </material>
   <material name="green">
-  	<color rgba="0 1 0 1"/>
+    <color rgba="0 1 0 1"/>
   </material>
   <material name="brown">
-  	<color rgba="0.65 0.16 0.16 1"/>
+    <color rgba="0.65 0.16 0.16 1"/>
   </material>
   <material name="violet">
-  	<color rgba="0.56 0 1 1"/>
+    <color rgba="0.56 0 1 1"/>
   </material>
 </robot>

File: description/urdf/urdf_final.urdf (robot description, URDF)
Before this commit: robot Mecanum_robot, 6 links, 5 joints
Links:
- added link lidar_frame; collision cylinder length=0.04 radius=0.05; visual cylinder length=0.04 radius=0.05
- link back_left_wheel_link: geometry collision mesh filename=/home/gunner/mecanum_robot/src/Mecanum_Robot_Simulation/des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; visual mesh filename=/home/gunner/mecanum_robot/src/Mecanum_Robot_Simulation/des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
- link back_right_wheel_link: geometry collision mesh filename=/home/gunner/mecanum_robot/src/Mecanum_Robot_Simulation/des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; visual mesh filename=/home/gunner/mecanum_robot/src/Mecanum_Robot_Simulation/des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
- link chasis: geometry collision mesh filename=/home/gunner/mecanum_robot/src/Mecanum_Robot_Simulation/des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; visual mesh filename=/home/gunner/mecanum_robot/src/Mecanum_Robot_Simulation/des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
- link front_left_wheel_link: geometry collision mesh filename=/home/gunner/mecanum_robot/src/Mecanum_Robot_Simulation/des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; visual mesh filename=/home/gunner/mecanum_robot/src/Mecanum_Robot_Simulation/des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
- link front_right_wheel_link: geometry collision mesh filename=/home/gunner/mecanum_robot/src/Mecanum_Robot_Simulation/des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; visual mesh filename=/home/gunner/mecanum_robot/src/Mecanum_Robot_Simulation/des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
Joints:
- added joint lidar_joint: type fixed, parent chasis, child lidar_frame, origin xyz=0 0 0 rpy=0 0 0
- joint back_left_wheel_joint: origin xyz=0.1175 -0.113 -0.03 rpy=-${math.pi/2} 0 ${math.pi} -> xyz=0.1175 -0.113 -0.03 rpy=-1.5708 0 3.1416
- joint back_right_wheel_joint: origin xyz=0.1175 0.113 -0.03 rpy=${math.pi/2} 0 ${math.pi} -> xyz=0.1175 0.113 -0.03 rpy=1.5708 0 3.1416
- joint front_left_wheel_joint: origin xyz=-0.1175 -0.113 -0.03 rpy=-${math.pi/2} 0 ${math.pi} -> xyz=-0.1175 -0.113 -0.03 rpy=-1.5708 0 3.1416
- joint front_right_wheel_joint: origin xyz=-0.1175 0.113 -0.03 rpy=${math.pi/2} 0 ${math.pi} -> xyz=-0.1175 0.113 -0.03 rpy=1.5708 0 3.1416
