Commit message: IMU position in visual fixed

File: description/urdf/gazeboIMU.xacro (robot description, xacro)
@@ -2,5 +2,5 @@
 <robot name="Mecanum_robot" xmlns:xacro="http://www.ros.org/wiki/xacro">
     <joint name="imu_joint" type="fixed">
-        <origin xyz="0 0 0.05" rpy="0 0 0"/> <!-- Positioned 0.05m above the lidar -->
+        <origin xyz="0 0 0.02" rpy="0 0 0"/> <!-- Positioned 0.05m above the lidar -->
         <parent link="lidar_frame"/>
         <child link="imu_link"/>

Commit message: Position of Lidar and IMU adjusted

File: description/urdf/gazeboIMU.xacro (robot description, xacro)
@@ -2,5 +2,5 @@
 <robot name="Mecanum_robot" xmlns:xacro="http://www.ros.org/wiki/xacro">
     <joint name="imu_joint" type="fixed">
-        <origin xyz="0 0 0.02" rpy="0 0 0"/> <!-- Positioned 0.05m above the lidar -->
+        <origin xyz="0 0 0.01" rpy="0 0 0"/> <!-- Positioned 0.05m above the lidar -->
         <parent link="lidar_frame"/>
         <child link="imu_link"/>

File: description/urdf/gazeboLidar.xacro (robot description, xacro)
@@ -11,5 +11,5 @@
   </xacro:macro>
   <joint name="lidar_joint" type="fixed">
-      <origin xyz="0 0 0" rpy="0 0 0" />
+      <origin xyz="0 0 0.01" rpy="0 0 0" />
       <parent link="chasis" />
       <child link="lidar_frame" />
@@ -18,5 +18,5 @@
     <visual>
       <geometry>
-        <cylinder radius="0.05" length="0.04"/>
+        <cylinder radius="0.05" length="0.02"/>
         <material name="red" />
       </geometry>
@@ -27,8 +27,8 @@
     <collision>
       <geometry>
-        <cylinder radius="0.05" length="0.04"/>
+        <cylinder radius="0.05" length="0.02"/>
       </geometry>
     </collision>
-    <xacro:inertial_cylinder mass="0.1" length="0.04" radius="0.05">
+    <xacro:inertial_cylinder mass="0.1" length="0.02" radius="0.05">
       <origin xyz="0 0 0" rpy="0 0 0"/>
     </xacro:inertial_cylinder>
