Commit message: Only rviz launcher problem remaining

File: description/urdf/gazebo_control.xacro (robot description, xacro)
@@ -13,5 +13,4 @@
         <plugin filename="gz-sim-joint-state-publisher-system" name="gz::sim::systems::JointStatePublisher">
             <topic>joint_states</topic>
-            <joint_name>base_footprint_joint</joint_name>
             <joint_name>back_right_wheel_joint</joint_name>
             <joint_name>back_left_wheel_joint</joint_name>
@@ -24,5 +23,5 @@
             <odom_topic>odometry</odom_topic>
             <tf_topic>tf</tf_topic>
-            <odom_publisher_frequency>50</odom_publisher_frequency>
+            <odom_publisher_frequency>30</odom_publisher_frequency>
         </plugin>
     </gazebo>

File: description/urdf/urdf_final.urdf (robot description, URDF)
Before this commit: robot Mecanum_robot, 7 links, 6 joints
Joints:
- joint base_footprint_joint: parent base_link -> chasis
