Commit message: added lidar

File: description/urdf/gazeboCamera.xacro (robot description, xacro)
@@ -1,21 +1,4 @@
 <?xml version="1.0"?>
 <robot xmlns:xacro="http://www.ros.org/wiki/xacro">
-    <gazebo>
-        <plugin name="gazebo_ros_joint_state_publisher"
-            filename="libgazebo_ros_joint_state_publisher.so">
-            <update_rate>20</update_rate>
-            <joint_name>chasis</joint_name>
-            <joint_name>back_right_wheel_joint</joint_name>
-            <joint_name>back_left_wheel_joint</joint_name>
-            <joint_name>front_right_wheel_joint</joint_name>
-            <joint_name>front_left_wheel_joint</joint_name>
-        </plugin>
-    </gazebo>
-    <gazebo>
-        <plugin name="gazebo_ros_joint_pose_trajectory"
-            filename="libgazebo_ros_joint_pose_trajectory.so">
-            <update_rate>20</update_rate>
-        </plugin>
-    </gazebo>
     <joint name="camera_optical_joint" type="fixed">
         <origin xyz="-0.25 0 0" rpy="0 0 ${math.pi}" />

File: description/urdf/material.xacro (robot description, xacro)
@@ -17,3 +17,3 @@
   	<color rgba="0.56 0 1 1"/>
   </material>
- </robot>
+</robot>

File: description/urdf/urdf_final.urdf (robot description, URDF)
Before this commit: robot Mecanum_robot, 6 links, 5 joints
Joints:
- joint back_left_wheel_joint: origin xyz=0.1175 -0.113 -0.03 rpy=-1.5708 -1.0094 3.1416 -> xyz=0.1175 -0.113 -0.03 rpy=-${math.pi/2} 0 ${math.pi}
- joint back_right_wheel_joint: origin xyz=0.1175 0.113 -0.03 rpy=1.5708 -0.55618 3.1416 -> xyz=0.1175 0.113 -0.03 rpy=${math.pi/2} 0 ${math.pi}
- joint front_left_wheel_joint: origin xyz=-0.1175 -0.113 -0.03 rpy=-1.5708 1.3416 3.1416 -> xyz=-0.1175 -0.113 -0.03 rpy=-${math.pi/2} 0 ${math.pi}
- joint front_right_wheel_joint: origin xyz=-0.1175 0.113 -0.03 rpy=1.5708 0.55618 3.1416 -> xyz=-0.1175 0.113 -0.03 rpy=${math.pi/2} 0 ${math.pi}

Commit message: Addednew sensors and features

File: description/urdf/gazeboCamera.xacro (robot description, xacro)
@@ -18,27 +18,31 @@
         <child link="camera_link_optical" />
     </joint>
-    <link name="camera_link_optical"></link>
-    <gazebo reference="camera_link">
-        <material>Gazebo/Red</material>
-        <sensor name="camera" type="camera">
-            <pose> 0 0 0 0 0 0 </pose>
-            <visualize>true</visualize>
-            <update_rate>10</update_rate>
-            <camera>
-                <horizontal_fov>1.089</horizontal_fov>
-                <image>
-                    <format>R8G8B8</format>
-                    <width>640</width>
-                    <height>480</height>
-                </image>
-                <clip>
-                    <near>0.05</near>
-                    <far>8.0</far>
-                </clip>
-            </camera>
-            <plugin name="camera_controller" filename="libgazebo_ros_camera.so">
-                <frame_name>camera_link_optical</frame_name>
-            </plugin>
-        </sensor>
-    </gazebo>
+    <link name="camera_link_optical">
+        <gazebo reference="camera_link">
+            <material>Gazebo/Red</material>
+            <sensor name="camera" type="camera">
+                <always_on>true</always_on>
+                <visualize>true</visualize>
+                <update_rate>30</update_rate>
+                <topic>camera/image_raw</topic>
+                <gz_frame_id>camera_rgb_frame</gz_frame_id>
+                <camera name="intel_realsense_r200">
+                <camera_info_topic>camera/camera_info</camera_info_topic>
+                    <horizontal_fov>1.089</horizontal_fov>
+                    <image>
+                        <format>R8G8B8</format>
+                        <width>640</width>
+                        <height>480</height>
+                    </image>
+                    <clip>
+                        <near>0.05</near>
+                        <far>8.0</far>
+                    </clip>
+                </camera>
+                <plugin name="camera_driver" filename="libgazebo_ros_camera.so">
+                    <frame_name>camera_link_optical</frame_name>
+                </plugin>
+            </sensor>
+        </gazebo>
+    </link>
 </robot>

File: description/urdf/gazeboLidar.xacro (robot description, xacro)
@@ -16,50 +16,55 @@
   </joint>
   <link name="lidar_frame">
-      <visual>
-          <geometry>
-              <cylinder radius="0.05" length="0.04"/>
-              <material name="brown" />
-          </geometry>
-      </visual>
-      <collision>
-          <geometry>
-              <cylinder radius="0.05" length="0.04"/>
-          </geometry>
-      </collision>
-      <xacro:inertial_cylinder mass="0.1" length="0.04" radius="0.05">
-          <origin xyz="0 0 0" rpy="0 0 0"/>
-      </xacro:inertial_cylinder>
+    <visual>
+      <geometry>
+        <cylinder radius="0.05" length="0.04"/>
+        <material name="red" />
+      </geometry>
+    </visual>
+    <collision>
+      <geometry>
+        <cylinder radius="0.05" length="0.04"/>
+      </geometry>
+    </collision>
+    <xacro:inertial_cylinder mass="0.1" length="0.04" radius="0.05">
+      <origin xyz="0 0 0" rpy="0 0 0"/>
+    </xacro:inertial_cylinder>
+    <gazebo reference="lidar_head_link">
+      <sensor name="lidar_head_link" type="gpu_lidar">
+        <always_on>true</always_on>
+        <visualize>true</visualize>
+        <pose relative_to='lidar_frame'>0 0 0 0 0 0</pose>
+        <update_rate>30</update_rate>
+        <gz_frame_id>lidar_head_link</gz_frame_id>
+        <topic>scan</topic>
+        <lidar>
+            <scan>
+                <horizontal>
+                    <samples>640</samples>
+                    <resolution>1</resolution>
+                    <min_angle>-1.396263</min_angle>
+                    <max_angle>1.396263</max_angle>
+                </horizontal>
+                <vertical>
+                    <samples>1</samples>
+                    <resolution>0.01</resolution>
+                    <min_angle>0</min_angle>
+                    <max_angle>0</max_angle>
+                </vertical>
+            </scan>
+            <range>
+                <min>0.08</min>
+                <max>10.0</max>
+                <resolution>0.01</resolution>
+            </range>
+            <frame_id>/lidar_head_link</frame_id>
+        </lidar>
+      </sensor>
+    </gazebo>
+    <gazebo>
+      <plugin filename="gz-sim-sensors-system" name="gz::sim::systems::Sensors">
+        <render_engine>ogre2</render_engine>
+      </plugin>
+    </gazebo>
   </link>
-  <gazebo>
-    <sensor name="lidar_head_link" type="gpu_lidar">
-      <update_rate>30</update_rate>
-      <lidar>
-        <scan>
-          <horizontal>
-            <samples>2800</samples>
-            <resolution>1</resolution>
-            <min_angle>-3.14</min_angle>
-            <max_angle>3.14</max_angle>
-          </horizontal>
-          <vertical>
-            <samples>1</samples>
-            <resolution>0.1</resolution>
-            <min_angle>0.0</min_angle>
-            <max_angle>0.0</max_angle>
-          </vertical>
-        </scan>
-        <range>
-          <min>0.2</min>
-          <max>30.0</max>
-          <resolution>0.01</resolution>
-        </range>
-      </lidar>
-      <always_on>true</always_on>
-      <visualize>true</visualize>
-      <pose>0 0 0.1 0 0 0</pose>  <!-- Adjust pose as needed -->
-    </sensor>
-    <plugin filename="gz-sim-sensors-system" name="gz::sim::systems::Sensors">
-      <render_engine>ogre2</render_engine>
-    </plugin>
-  </gazebo>
 </robot>

File: description/urdf/gazeboTransforms_update.xacro (robot description, xacro)
@@ -2,7 +2,5 @@
 <robot xmlns:xacro="http://www.ros.org/wiki/xacro">
     <gazebo>
-        <plugin name="gazebo_ros_joint_state_publisher"
-            filename="libgazebo_ros_joint_state_publisher.so">
-            <update_rate>20</update_rate>
+        <plugin filename="gz-sim-joint-state-publisher-system" name="gz::sim::systems::JointStatePublisher">
             <joint_name>chasis_joint</joint_name>
             <joint_name>back_right_wheel_joint</joint_name>
@@ -12,9 +10,9 @@
         </plugin>
     </gazebo>
-    <gazebo>
+    <!-- <gazebo>
         <plugin name="gazebo_ros_joint_pose_trajectory"
             filename="libgazebo_ros_joint_pose_trajectory.so">
             <update_rate>20</update_rate>
         </plugin>
-    </gazebo>
+    </gazebo> -->
 </robot>

File: description/urdf/urdf_final.urdf (robot description, URDF)
Before this commit: robot Mecanum_robot, 7 links, 6 joints
Links:
- removed link lidar_frame
- link back_left_wheel_link: geometry collision mesh filename=$(find mecanum_robot_simulation)/description/meshes/back_le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; visual mesh filename=$(find mecanum_robot_simulation)/description/meshes/back_le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
- link back_right_wheel_link: geometry collision mesh filename=$(find mecanum_robot_simulation)/description/meshes/back_ri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; visual mesh filename=$(find mecanum_robot_simulation)/description/meshes/back_ri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
- link chasis: geometry collision mesh filename=$(find mecanum_robot_simulation)/description/meshes/chasis.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; visual mesh filename=$(find mecanum_robot_simulation)/description/meshes/chasis.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
- link front_left_wheel_link: geometry collision mesh filename=$(find mecanum_robot_simulation)/description/meshes/front_l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; visual mesh filename=$(find mecanum_robot_simulation)/description/meshes/front_l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
- link front_right_wheel_link: geometry collision mesh filename=$(find mecanum_robot_simulation)/description/meshes/front_r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; visual mesh filename=$(find mecanum_robot_simulation)/description/meshes/front_r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
Joints:
- removed joint lidar_joint

Commit message: Robot launchd in rviz though comicallz

File: description/urdf/gazeboCamera.xacro (robot description, xacro)
@@ -21,26 +21,21 @@
         <gazebo reference="camera_link">
             <material>Gazebo/Red</material>
-            <sensor name="camera" type="camera">
-                <always_on>true</always_on>
-                <visualize>true</visualize>
-                <update_rate>30</update_rate>
-                <topic>camera/image_raw</topic>
-                <gz_frame_id>camera_rgb_frame</gz_frame_id>
-                <camera name="intel_realsense_r200">
-                <camera_info_topic>camera/camera_info</camera_info_topic>
-                    <horizontal_fov>1.089</horizontal_fov>
+            <sensor name="rgbd_camera" type="rgbd_camera">
+                <camera>
+                    <horizontal_fov>1.047</horizontal_fov>
                     <image>
-                        <format>R8G8B8</format>
-                        <width>640</width>
-                        <height>480</height>
+                      <width>320</width>
+                      <height>240</height>
                     </image>
                     <clip>
-                        <near>0.05</near>
-                        <far>8.0</far>
+                      <near>0.1</near>
+                      <far>100</far>
                     </clip>
                 </camera>
-                <plugin name="camera_driver" filename="libgazebo_ros_camera.so">
-                    <frame_name>camera_link_optical</frame_name>
-                </plugin>
+                <always_on>1</always_on>
+                <update_rate>30</update_rate>
+                <visualize>true</visualize>
+                <topic>rgbd_camera</topic>
+                <plugin filename="RosGzPointCloud" name="ros_gz_point_cloud::PointCloud" />
             </sensor>
         </gazebo>

File: description/urdf/gazeboDepthCamera.xacro (robot description, xacro)
@@ -21,30 +21,26 @@
     <gazebo reference="camera_link">
         <material>Gazebo/Red</material>
-        <sensor type="depth" name="my_camera">
-            <update_rate>20</update_rate>
+        <sensor name="depth_camera" type="depth_camera">
+            <camera>
+              <horizontal_fov>1.047</horizontal_fov>
+              <image>
+                <width>320</width>
+                <height>240</height>
+                <format>R_FLOAT32</format>
+              </image>
+              <clip>
+                <near>0.1</near>
+                <far>100</far>
+              </clip>
+            </camera>
+            <always_on>1</always_on>
+            <update_rate>10</update_rate>
             <visualize>true</visualize>
-            <camera name="cam">
-                <horizontal_fov>1.089</horizontal_fov>
-                <image>
-                    <width>640</width>
-                    <height>480</height>
-                    <format>B8G8R8</format>
-                </image>
-                <clip>
-                    <near>0.05</near>
-                    <far>8.0</far>
-                </clip>
-                <noise>
-                    <type>gaussian</type>
-                    <mean>0.0</mean>
-                    <stddev>0.007</stddev>
-                </noise>
-            </camera>
-            <plugin name="camera_controller" filename="libgazebo_ros_camera.so">
-                <frame_name>camera_link_optical</frame_name>
-                <min_depth>0.1</min_depth>
-                <max_depth>500</max_depth>
+            <topic>depth_camera</topic>
+            <plugin filename="RosGzPointCloud" name="ros_gz_point_cloud::PointCloud">
+              <topic>points</topic>
+              <frame_id>map</frame_id>
             </plugin>
-        </sensor>
+          </sensor>
     </gazebo>
 </robot>

File: description/urdf/gazeboLidar.xacro (robot description, xacro)
@@ -30,40 +30,37 @@
       <origin xyz="0 0 0" rpy="0 0 0"/>
     </xacro:inertial_cylinder>
-    <gazebo reference="lidar_head_link">
-      <sensor name="lidar_head_link" type="gpu_lidar">
-        <always_on>true</always_on>
+    <gazebo reference="lidar_frame">
+      <sensor name='gpu_lidar' type='gpu_lidar'>
+        <topic>lidar</topic> <!-- Ensure this matches the output from `gz topic -l` -->
+        <update_rate>10</update_rate>
+        <lidar>
+          <scan>
+            <horizontal>
+              <samples>640</samples>
+              <resolution>1</resolution>
+              <min_angle>-1.396263</min_angle>
+              <max_angle>1.396263</max_angle>
+            </horizontal>
+            <vertical>
+              <samples>16</samples>
+              <resolution>1</resolution>
+              <min_angle>-0.261799</min_angle>
+              <max_angle>0.261799</max_angle>
+            </vertical>
+          </scan>
+          <range>
+            <min>0.08</min>
+            <max>10.0</max>
+            <resolution>0.01</resolution>
+          </range>
+        </lidar>
+        <alwaysOn>1</alwaysOn>
         <visualize>true</visualize>
-        <pose relative_to='lidar_frame'>0 0 0 0 0 0</pose>
-        <update_rate>30</update_rate>
-        <gz_frame_id>lidar_head_link</gz_frame_id>
-        <topic>scan</topic>
-        <lidar>
-            <scan>
-                <horizontal>
-                    <samples>640</samples>
-                    <resolution>1</resolution>
-                    <min_angle>-1.396263</min_angle>
-                    <max_angle>1.396263</max_angle>
-                </horizontal>
-                <vertical>
-                    <samples>1</samples>
-                    <resolution>0.01</resolution>
-                    <min_angle>0</min_angle>
-                    <max_angle>0</max_angle>
-                </vertical>
-            </scan>
-            <range>
-                <min>0.08</min>
-                <max>10.0</max>
-                <resolution>0.01</resolution>
-            </range>
-            <frame_id>/lidar_head_link</frame_id>
-        </lidar>
+        <plugin filename="RosGzPointCloud" name="ros_gz_point_cloud::PointCloud">
+          <namespace>custom_params</namespace>
+          <topic>pc2</topic> <!-- This topic is for point cloud data -->
+          <frame_id>lidar_frame</frame_id> <!-- Make sure this matches the actual frame name -->
+        </plugin>
       </sensor>
-    </gazebo>
-    <gazebo>
-      <plugin filename="gz-sim-sensors-system" name="gz::sim::systems::Sensors">
-        <render_engine>ogre2</render_engine>
-      </plugin>
     </gazebo>
   </link>

File: description/urdf/urdf_final.urdf (robot description, URDF)
Before this commit: robot Mecanum_robot, 6 links, 5 joints
Links:
- link back_left_wheel_link: geometry collision cylinder length=0.039 radius=0.029; visual mesh filename=file:///home/gunner/mecanum_robot/src/mecanum_robot_simulat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
- link back_right_wheel_link: geometry collision cylinder length=0.039 radius=0.029; visual mesh filename=file:///home/gunner/mecanum_robot/src/mecanum_robot_simulat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
- link chasis: geometry collision box size=0.50 0.40 0.05; visual mesh filename=file:///home/gunner/mecanum_robot/src/mecanum_robot_simulat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
- link front_left_wheel_link: geometry collision cylinder length=0.039 radius=0.029; visual mesh filename=file:///home/gunner/mecanum_robot/src/mecanum_robot_simulat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
- link front_right_wheel_link: geometry collision cylinder length=0.039 radius=0.029; visual mesh filename=file:///home/gunner/mecanum_robot/src/mecanum_robot_simulat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
