Commit message: Can be seen in rviz and control implemented

File: description/urdf/gazeboCamera.xacro (robot description, xacro)
@@ -11,4 +11,7 @@
                 <box size="0.010 0.03 0.03"/>
             </geometry>
+            <material name="red">
+                <color rgba="1 0 0 1"/>
+            </material>
         </visual>
     </link>
@@ -20,23 +23,28 @@
     <link name="camera_link_optical">
         <gazebo reference="camera_link">
-            <material>Gazebo/Red</material>
-            <sensor name="rgbd_camera" type="rgbd_camera">
-                <camera>
-                    <horizontal_fov>1.047</horizontal_fov>
-                    <image>
-                      <width>320</width>
-                      <height>240</height>
-                    </image>
-                    <clip>
-                      <near>0.1</near>
-                      <far>100</far>
-                    </clip>
-                </camera>
-                <always_on>1</always_on>
-                <update_rate>30</update_rate>
-                <visualize>true</visualize>
-                <topic>rgbd_camera</topic>
-                <plugin filename="RosGzPointCloud" name="ros_gz_point_cloud::PointCloud" />
-            </sensor>
+          <material>Gazebo/Red</material>
+          <sensor name="camera" type="camera">
+            <always_on>true</always_on>
+            <visualize>true</visualize>
+            <update_rate>30</update_rate>
+            <topic>camera/image_raw</topic>
+            <gz_frame_id>camera_link_optical</gz_frame_id>
+            <camera name="intel_realsense_r200">
+              <camera_info_topic>camera/camera_info</camera_info_topic>
+              <horizontal_fov>1.089</horizontal_fov>
+              <image>
+                <format>R8G8B8</format>
+                <width>640</width>
+                <height>480</height>
+              </image>
+              <clip>
+                <near>0.05</near>
+                <far>8.0</far>
+              </clip>
+            </camera>
+            <plugin filename="libgazebo_ros_camera.so" name="camera_driver">
+              <frame_name>camera_link_optical</frame_name>
+            </plugin>
+          </sensor>
         </gazebo>
     </link>

File: description/urdf/gazeboLidar.xacro (robot description, xacro)
@@ -21,4 +21,7 @@
         <material name="red" />
       </geometry>
+      <material name="red">
+        <color rgba="1 0 0 1"/>
+      </material>
     </visual>
     <collision>
@@ -30,36 +33,34 @@
       <origin xyz="0 0 0" rpy="0 0 0"/>
     </xacro:inertial_cylinder>
-    <gazebo reference="lidar_frame">
-      <sensor name='gpu_lidar' type='gpu_lidar'>
-        <topic>lidar</topic> <!-- Ensure this matches the output from `gz topic -l` -->
-        <update_rate>10</update_rate>
+    <gazebo reference="lidar_head_link" >
+      <sensor name="lidar_head_link" type="gpu_lidar">
+        <gz_frame_id>lidar_head_link</gz_frame_id>
+        <topic>scan</topic>
+        <update_rate>30</update_rate>
+        <!-- <plugin filename="gz::sim::lidar" name="lidar"></plugin> -->
         <lidar>
           <scan>
             <horizontal>
-              <samples>640</samples>
+              <samples>2800</samples>
               <resolution>1</resolution>
-              <min_angle>-1.396263</min_angle>
-              <max_angle>1.396263</max_angle>
+              <min_angle>-3.14</min_angle>
+              <max_angle>3.14</max_angle>
             </horizontal>
             <vertical>
-              <samples>16</samples>
-              <resolution>1</resolution>
-              <min_angle>-0.261799</min_angle>
-              <max_angle>0.261799</max_angle>
+              <samples>1</samples>
+              <resolution>0.1</resolution>
+              <min_angle>0.0</min_angle>
+              <max_angle>0.0</max_angle>
             </vertical>
           </scan>
           <range>
-            <min>0.08</min>
-            <max>10.0</max>
+            <min>0.2</min>
+            <max>30.0</max>
             <resolution>0.01</resolution>
           </range>
+          <frame_id>/lidar_head_link</frame_id>
         </lidar>
-        <alwaysOn>1</alwaysOn>
+        <alwaysOn>ture</alwaysOn>
         <visualize>true</visualize>
-        <plugin filename="RosGzPointCloud" name="ros_gz_point_cloud::PointCloud">
-          <namespace>custom_params</namespace>
-          <topic>pc2</topic> <!-- This topic is for point cloud data -->
-          <frame_id>lidar_frame</frame_id> <!-- Make sure this matches the actual frame name -->
-        </plugin>
       </sensor>
     </gazebo>

File: description/urdf/gazeboTransforms_update.xacro (robot description, xacro)
@@ -3,4 +3,5 @@
     <gazebo>
         <plugin filename="gz-sim-joint-state-publisher-system" name="gz::sim::systems::JointStatePublisher">
+            <topic>joint_states</topic>
             <joint_name>chasis_joint</joint_name>
             <joint_name>back_right_wheel_joint</joint_name>
@@ -10,9 +11,3 @@
         </plugin>
     </gazebo>
-    <!-- <gazebo>
-        <plugin name="gazebo_ros_joint_pose_trajectory"
-            filename="libgazebo_ros_joint_pose_trajectory.so">
-            <update_rate>20</update_rate>
-        </plugin>
-    </gazebo> -->
 </robot>

File: description/urdf/gazebo_control.xacro (robot description, xacro)
@@ -2,16 +2,12 @@
 <robot xmlns:xacro="http://www.ros.org/wiki/xacro">
     <gazebo>
-        <plugin name="robot_control" filename="libgazebo_ros_diff_drive.so">
-            <left_joint>back_left_wheel_joint</left_joint>
-            <right_joint>back_right_wheel_joint</right_joint>
+        <plugin name="gz::sim::systems::MecanumDrive" filename="gz-sim-mecanum-drive-system">
+            <front_left_joint>front_left_wheel_joint</front_left_joint>
+            <front_right_joint>front_right_wheel_joint</front_right_joint>
+            <back_left_joint>back_left_wheel_joint</back_left_joint>
+            <back_right_joint>back_right_wheel_joint</back_right_joint>
             <wheel_separation>0.226</wheel_separation>
-            <wheel_diameter>0.058</wheel_diameter>
-            <wheel_torque>5.0</wheel_torque>
-            <max_wheel_acceleration>10.0</max_wheel_acceleration>
-            <odometry_frame>odom</odometry_frame>
-            <robot_base_frame>base_link</robot_base_frame>
-            <publish_odom>true</publish_odom>
-            <publish_odom_tf>true</publish_odom_tf>
-            <publish_wheel_tf>true</publish_wheel_tf>
+            <wheel_radius>0.029</wheel_radius>
+            <wheelbase>0.235</wheelbase>
         </plugin>
     </gazebo>

Commit message: Lidar and IMU sensors in working condition

File: description/urdf/gazeboCamera.xacro (robot description, xacro)
@@ -24,10 +24,10 @@
         <gazebo reference="camera_link">
           <material>Gazebo/Red</material>
-          <sensor name="camera" type="camera">
+          <sensor name="IMX219" type="camera">
             <always_on>true</always_on>
             <visualize>true</visualize>
             <update_rate>30</update_rate>
             <topic>camera/image_raw</topic>
-            <gz_frame_id>camera_link_optical</gz_frame_id>
+            <gz_frame_id>camera_rgb_frame</gz_frame_id>
             <camera name="intel_realsense_r200">
               <camera_info_topic>camera/camera_info</camera_info_topic>
@@ -43,7 +43,4 @@
               </clip>
             </camera>
-            <plugin filename="libgazebo_ros_camera.so" name="camera_driver">
-              <frame_name>camera_link_optical</frame_name>
-            </plugin>
           </sensor>
         </gazebo>

File: description/urdf/gazeboLidar.xacro (robot description, xacro)
@@ -33,36 +33,38 @@
       <origin xyz="0 0 0" rpy="0 0 0"/>
     </xacro:inertial_cylinder>
-    <gazebo reference="lidar_head_link" >
-      <sensor name="lidar_head_link" type="gpu_lidar">
-        <gz_frame_id>lidar_head_link</gz_frame_id>
-        <topic>scan</topic>
-        <update_rate>30</update_rate>
-        <!-- <plugin filename="gz::sim::lidar" name="lidar"></plugin> -->
-        <lidar>
+  </link>
+  <gazebo>
+    <plugin filename="gz-sim-sensors-system" name="gz::sim::systems::Sensors">
+      <render_engine>ogre2</render_engine>
+    </plugin>
+  </gazebo>
+  <gazebo reference="lidar_frame" >
+    <sensor name="lidar_frame" type="gpu_lidar">
+      <topic>lidar</topic>
+      <update_rate>10</update_rate>
+      <ray>
           <scan>
-            <horizontal>
-              <samples>2800</samples>
-              <resolution>1</resolution>
-              <min_angle>-3.14</min_angle>
-              <max_angle>3.14</max_angle>
-            </horizontal>
-            <vertical>
-              <samples>1</samples>
-              <resolution>0.1</resolution>
-              <min_angle>0.0</min_angle>
-              <max_angle>0.0</max_angle>
-            </vertical>
+              <horizontal>
+                  <samples>640</samples>
+                  <resolution>1</resolution>
+                  <min_angle>-1.396263</min_angle>
+                  <max_angle>1.396263</max_angle>
+              </horizontal>
+              <vertical>
+                  <samples>1</samples>
+                  <resolution>0.01</resolution>
+                  <min_angle>0</min_angle>
+                  <max_angle>0</max_angle>
+              </vertical>
           </scan>
           <range>
-            <min>0.2</min>
-            <max>30.0</max>
-            <resolution>0.01</resolution>
+              <min>0.08</min>
+              <max>10.0</max>
+              <resolution>0.01</resolution>
           </range>
-          <frame_id>/lidar_head_link</frame_id>
-        </lidar>
-        <alwaysOn>ture</alwaysOn>
-        <visualize>true</visualize>
-      </sensor>
-    </gazebo>
-  </link>
+      </ray>
+      <always_on>1</always_on>
+      <visualize>true</visualize>
+    </sensor>
+  </gazebo>
 </robot>

Commit message: All working according to plan

File: description/urdf/gazeboCamera.xacro (robot description, xacro)
@@ -1,48 +1,47 @@
 <?xml version="1.0"?>
 <robot xmlns:xacro="http://www.ros.org/wiki/xacro">
-    <joint name="camera_joint" type="fixed">
-        <origin xyz="-0.255 0 -0.015" rpy="0 0 ${math.pi}" />
-        <parent link="chasis" />
-        <child link="camera_link" />
-    </joint>
-    <link name="camera_link">
-        <visual>
-            <geometry>
-                <box size="0.010 0.03 0.03"/>
-            </geometry>
-            <material name="red">
-                <color rgba="1 0 0 1"/>
-            </material>
-        </visual>
-    </link>
-    <joint name="camera_optical_joint" type="fixed">
-        <origin xyz="0 0 0" rpy="${-math.pi/2} 0 ${-math.pi/22}" />
-        <parent link="camera_link" />
-        <child link="camera_link_optical" />
-    </joint>
-    <link name="camera_link_optical">
-        <gazebo reference="camera_link">
-          <material>Gazebo/Red</material>
-          <sensor name="IMX219" type="camera">
-            <always_on>true</always_on>
-            <visualize>true</visualize>
-            <update_rate>30</update_rate>
-            <topic>camera/image_raw</topic>
-            <gz_frame_id>camera_rgb_frame</gz_frame_id>
-            <camera name="intel_realsense_r200">
-              <camera_info_topic>camera/camera_info</camera_info_topic>
-              <horizontal_fov>1.089</horizontal_fov>
-              <image>
-                <format>R8G8B8</format>
-                <width>640</width>
-                <height>480</height>
-              </image>
-              <clip>
-                <near>0.05</near>
-                <far>8.0</far>
-              </clip>
-            </camera>
-          </sensor>
-        </gazebo>
-    </link>
+  <joint name="camera_joint" type="fixed">
+      <origin xyz="-0.255 0 -0.015" rpy="0 0 ${math.pi}" />
+      <parent link="chasis" />
+      <child link="camera_link" />
+  </joint>
+  <link name="camera_link">
+      <visual>
+          <geometry>
+              <box size="0.010 0.03 0.03"/>
+          </geometry>
+          <material name="red">
+              <color rgba="1 0 0 1"/>
+          </material>
+      </visual>
+  </link>
+  <joint name="camera_optical_joint" type="fixed">
+      <origin xyz="0 0 0" rpy="${-math.pi/2} 0 ${-math.pi/22}" />
+      <parent link="camera_link" />
+      <child link="camera_link_optical" />
+  </joint>
+  <link name="camera_link_optical"></link>
+  <gazebo reference="camera_link">
+    <material>Gazebo/Red</material>
+    <sensor name="camera" type="camera">
+      <pose> 0 0 0 0 0 0 </pose>
+      <visualize>true</visualize>
+      <update_rate>10</update_rate>
+      <camera>
+          <camera_info_topic>camera/camera_info</camera_info_topic>
+          <horizontal_fov>1.089</horizontal_fov>
+          <image>
+              <format>R8G8B8</format>
+              <width>640</width>
+              <height>480</height>
+          </image>
+          <clip>
+              <near>0.05</near>
+              <far>8.0</far>
+          </clip>
+      </camera>
+      <topic>camera/image_raw</topic>
+      <gz_frame_id>camera_link_optical</gz_frame_id>
+    </sensor>
+  </gazebo>
 </robot>

File: description/urdf/gazeboIMU.xacro (robot description, xacro)
@@ -1,39 +1,40 @@
 <?xml version="1.0"?>
 <robot name="Mecanum_robot" xmlns:xacro="http://www.ros.org/wiki/xacro">
-    <joint name="imu_joint" type="fixed">
-        <origin xyz="0 0 0.01" rpy="0 0 0"/> <!-- Positioned 0.05m above the lidar -->
-        <parent link="lidar_frame"/>
-        <child link="imu_link"/>
-    </joint>
-    <link name="imu_link">
-        <inertial>
-          <mass value="0.01"/> <!-- Adjust this based on the actual weight of the IMU -->
-          <origin xyz="0 0 0" rpy="0 0 0"/>
-          <inertia ixx="0.0001" ixy="0.0" ixz="0.0" iyy="0.0001" iyz="0.0" izz="0.0001"/>
-        </inertial>
-        <visual>
-          <geometry>
-            <box size="0.03 0.03 0.01"/> <!-- Size of the IMU -->
-          </geometry>
-          <material name="grey">
-            <color rgba="0.5 0.5 0.5 1"/>
-          </material>
-        </visual>
-        <collision>
-          <geometry>
-            <box size="0.03 0.03 0.01"/> <!-- Same size for collision geometry -->
-          </geometry>
-        </collision>
-    </link>
-    <gazebo>
-        <plugin filename="gz-sim-imu-system" name="gz::sim::systems::Imu" />
-    </gazebo>
-    <gazebo reference="imu_link">
-        <sensor name="imu_sensor" type="imu">
-            <always_on>1</always_on>
-            <update_rate>1</update_rate>
-            <visualize>true</visualize>
-            <topic>imu</topic>
-        </sensor>
-    </gazebo>
+  <joint name="imu_joint" type="fixed">
+      <origin xyz="0 0 0.01" rpy="0 0 0"/> <!-- Positioned 0.05m above the lidar -->
+      <parent link="lidar_frame"/>
+      <child link="imu_link"/>
+  </joint>
+  <link name="imu_link">
+      <inertial>
+        <mass value="0.01"/> <!-- Adjust this based on the actual weight of the IMU -->
+        <origin xyz="0 0 0" rpy="0 0 0"/>
+        <inertia ixx="0.0001" ixy="0.0" ixz="0.0" iyy="0.0001" iyz="0.0" izz="0.0001"/>
+      </inertial>
+      <visual>
+        <geometry>
+          <box size="0.03 0.03 0.01"/> <!-- Size of the IMU -->
+        </geometry>
+        <material name="grey">
+          <color rgba="0.5 0.5 0.5 1"/>
+        </material>
+      </visual>
+      <collision>
+        <geometry>
+          <box size="0.03 0.03 0.01"/> <!-- Same size for collision geometry -->
+        </geometry>
+      </collision>
+  </link>
+  <gazebo>
+    <plugin filename="gz-sim-imu-system" name="gz::sim::systems::Imu" />
+  </gazebo>
+  <gazebo reference="imu_link">
+    <sensor name="imu_sensor" type="imu">
+      <always_on>1</always_on>
+      <update_rate>1</update_rate>
+      <visualize>true</visualize>
+      <topic>imu</topic>
+      <gz_frame_id>imu_link</gz_frame_id>
+    </sensor>
+  </gazebo>
 </robot>

File: description/urdf/gazeboLidar.xacro (robot description, xacro)
@@ -40,30 +40,31 @@
   </gazebo>
   <gazebo reference="lidar_frame" >
-    <sensor name="lidar_frame" type="gpu_lidar">
-      <topic>lidar</topic>
-      <update_rate>10</update_rate>
-      <ray>
-          <scan>
-              <horizontal>
-                  <samples>640</samples>
-                  <resolution>1</resolution>
-                  <min_angle>-1.396263</min_angle>
-                  <max_angle>1.396263</max_angle>
-              </horizontal>
-              <vertical>
-                  <samples>1</samples>
-                  <resolution>0.01</resolution>
-                  <min_angle>0</min_angle>
-                  <max_angle>0</max_angle>
-              </vertical>
-          </scan>
-          <range>
-              <min>0.08</min>
-              <max>10.0</max>
-              <resolution>0.01</resolution>
-          </range>
-      </ray>
+    <sensor name="laser" type="gpu_lidar">
+      <topic>scan</topic>
+      <update_rate>30</update_rate>
+      <lidar>
+        <scan>
+          <horizontal>
+            <samples>2800</samples>
+            <resolution>1</resolution>
+            <min_angle>-3.14</min_angle>
+            <max_angle>3.14</max_angle>
+          </horizontal>
+          <vertical>
+            <samples>1</samples>
+            <resolution>0.1</resolution>
+            <min_angle>0.0</min_angle>
+            <max_angle>0.0</max_angle>
+          </vertical>
+        </scan>
+        <range>
+          <min>0.2</min>
+          <max>30.0</max>
+          <resolution>0.01</resolution>
+        </range>
+      </lidar>
       <always_on>1</always_on>
       <visualize>true</visualize>
+      <gz_frame_id>lidar_frame</gz_frame_id>
     </sensor>
   </gazebo>

Commit message: Added slam and all required things

File: description/urdf/gazeboCamera.xacro (robot description, xacro)
@@ -25,5 +25,5 @@
     <material>Gazebo/Red</material>
     <sensor name="camera" type="camera">
-      <pose> 0 0 0 0 0 0 </pose>
+      <pose> 0 0 0 0 -1.57 0 </pose>
       <visualize>true</visualize>
       <update_rate>10</update_rate>

File: description/urdf/gazeboTransforms_update.xacro (robot description, xacro)
@@ -4,5 +4,4 @@
         <plugin filename="gz-sim-joint-state-publisher-system" name="gz::sim::systems::JointStatePublisher">
             <topic>joint_states</topic>
-            <joint_name>chasis_joint</joint_name>
             <joint_name>back_right_wheel_joint</joint_name>
             <joint_name>back_left_wheel_joint</joint_name>

File: description/urdf/gazebo_control.xacro (robot description, xacro)
@@ -10,4 +10,10 @@
             <wheel_radius>0.029</wheel_radius>
             <wheelbase>0.235</wheelbase>
+            <!-- Set the odometry frame and child frame -->
+            <tf_topic>model/mecanum_robot/tf</tf_topic>
+            <frame_id>odom</frame_id>             <!-- Odometry frame -->
+            <child_frame_id>base_link</child_frame_id>  <!-- Robot's base frame -->
+            <!-- Optional: set odometry publish frequency -->
+            <odom_publish_frequency>50</odom_publish_frequency>  <!-- Adjust as needed -->
         </plugin>
     </gazebo>

File: description/urdf/urdf_final.urdf (robot description, URDF)
Before this commit: robot Mecanum_robot, 6 links, 5 joints
Links:
- added link base_footprint_link; visual box size=0.235 0.226 0.001
Joints:
- added joint base_footprint_joint: type fixed, parent base_link, child base_footprint_link, origin xyz=0 0 0 rpy=0 0 0

Commit message: Mainly changed the nav2 params file

File: description/urdf/gazeboCamera.xacro (robot description, xacro)
@@ -17,5 +17,5 @@
   </link>
   <joint name="camera_optical_joint" type="fixed">
-      <origin xyz="0 0 0" rpy="${-math.pi/2} 0 ${-math.pi/22}" />
+      <origin xyz="0 0 0" rpy="${-math.pi/2} 0 0" />
       <parent link="camera_link" />
       <child link="camera_link_optical" />
@@ -25,20 +25,20 @@
     <material>Gazebo/Red</material>
     <sensor name="camera" type="camera">
-      <pose> 0 0 0 0 -1.57 0 </pose>
-      <visualize>true</visualize>
-      <update_rate>10</update_rate>
-      <camera>
-          <camera_info_topic>camera/camera_info</camera_info_topic>
-          <horizontal_fov>1.089</horizontal_fov>
-          <image>
-              <format>R8G8B8</format>
-              <width>640</width>
-              <height>480</height>
-          </image>
-          <clip>
-              <near>0.05</near>
-              <far>8.0</far>
-          </clip>
-      </camera>
+        <pose> 0 0 0 0 0 0 </pose>
+        <visualize>true</visualize>
+        <update_rate>10</update_rate>
+        <camera>
+            <camera_info_topic>camera/camera_info</camera_info_topic>
+            <horizontal_fov>1.089</horizontal_fov>
+            <image>
+                <format>R8G8B8</format>
+                <width>640</width>
+                <height>480</height>
+            </image>
+            <clip>
+                <near>0.05</near>
+                <far>8.0</far>
+            </clip>
+        </camera>
       <topic>camera/image_raw</topic>
       <gz_frame_id>camera_link_optical</gz_frame_id>

File: description/urdf/urdf_final.urdf (robot description, URDF)
Before this commit: robot Mecanum_robot, 7 links, 6 joints
Joints:
- joint chasis_joint: origin xyz=0 0 0 rpy=0 0 0 -> xyz=0 0 0 rpy=0 0 3.14
