Commit message: Adjusted the joints axes

File: description/urdf/gazeboCamera.xacro (robot description, xacro)
@@ -2,5 +2,5 @@
 <robot xmlns:xacro="http://www.ros.org/wiki/xacro">
   <joint name="camera_joint" type="fixed">
-      <origin xyz="-0.255 0 -0.015" rpy="0 0 ${math.pi}" />
+      <origin xyz="0.255 0 -0.015" rpy="0 0 0" />
       <parent link="chasis" />
       <child link="camera_link" />
@@ -17,5 +17,5 @@
   </link>
   <joint name="camera_optical_joint" type="fixed">
-      <origin xyz="0 0 0" rpy="${-math.pi/2} 0 0" />
+      <origin xyz="0 0 0" rpy="-1.5708 0 -1.5708" />
       <parent link="camera_link" />
       <child link="camera_link_optical" />

File: description/urdf/urdf_final.urdf (robot description, URDF)
Before this commit: robot Mecanum_robot, 7 links, 6 joints
Joints:
- joint back_left_wheel_joint: limit lower=-3.14 upper=3.14 effort=200 velocity=5 -> lower=-3.14 upper=3.14 effort=200 velocity=15; origin xyz=0.1175 -0.113 -0.03 rpy=-1.5708 0 3.1416 -> xyz=-0.1175 0.113 -0.03 rpy=1.5708 0 3.1416
- joint back_right_wheel_joint: limit lower=-3.14 upper=3.14 effort=200 velocity=5 -> lower=-3.14 upper=3.14 effort=200 velocity=15; origin xyz=0.1175 0.113 -0.03 rpy=1.5708 0 3.1416 -> xyz=-0.1175 -0.113 -0.03 rpy=-1.5708 0 -3.1416
- joint chasis_joint: origin xyz=0 0 0 rpy=0 0 3.14 -> xyz=0 0 0 rpy=0 0 3.1416
- joint front_left_wheel_joint: limit lower=-3.14 upper=3.14 effort=200 velocity=5 -> lower=-3.14 upper=3.14 effort=200 velocity=15; origin xyz=-0.1175 -0.113 -0.03 rpy=-1.5708 0 3.1416 -> xyz=0.1175 0.113 -0.03 rpy=1.5708 0 3.1416
- joint front_right_wheel_joint: limit lower=-3.14 upper=3.14 effort=200 velocity=5 -> lower=-3.14 upper=3.14 effort=200 velocity=15; origin xyz=-0.1175 0.113 -0.03 rpy=1.5708 0 3.1416 -> xyz=0.1175 -0.113 -0.03 rpy=-1.5708 0 3.1416
