Commit message: No big error in Gazebo launch

File: description/urdf/urdf_final.urdf (robot description, URDF)
Before this commit: robot Mecanum_robot, 6 links, 5 joints
Links:
- link back_left_wheel_link: geometry collision cylinder length=0.039 radius=0.029; visual mesh filename=package://mecanum_robot_simulation/description/meshes/back_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
- link back_right_wheel_link: geometry collision cylinder length=0.039 radius=0.029; visual mesh filename=package://mecanum_robot_simulation/description/meshes/back_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
- link base_link: mass None -> 0.1; geometry collision box size=0.01 0.01 0.01
- link chasis: geometry collision box size=0.50 0.40 0.05; visual mesh filename=package://mecanum_robot_simulation/description/meshes/chasi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
- link front_left_wheel_link: geometry collision cylinder length=0.039 radius=0.029; visual mesh filename=package://mecanum_robot_simulation/description/meshes/front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
- link front_right_wheel_link: geometry collision cylinder length=0.039 radius=0.029; visual mesh filename=package://mecanum_robot_simulation/description/meshes/front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

Commit message: Corrected the transform tree

File: description/urdf/urdf_final.urdf (robot description, URDF)
Before this commit: robot Mecanum_robot, 7 links, 6 joints
Joints:
- joint chasis_joint: origin xyz=0 0 0 rpy=0 0 3.1416 -> xyz=0 0 0 rpy=0 0 0
